File: Minilab/Entradas-salidas/entrada.kicad_pcb (KiCad board)
At the start: 2 copper layers, 70.6 x 51.2 mm, 66 parts, among them J1 Out 5V/0V, J10 Vin, J11 Vin, J12 Vin, J13 Vin, J14 Conn_01x10_Pin, J15 Vin, J16 Vin, J2 Out 5V/0V, J3 Out 5V/0V, J4 Out 5V/0V, J5 Out 5V/0V, J6 Out 5V/0V, J7 Vin, J8 Vin, J9 Vin, SW1 SW_SPST, SW2 SW_SPST, SW3 SW_SPST, SW4 SW_SPST, SW5 SW_SPST, SW6 SW_SPST, U1 4049, U10 NE555P, U2 Mini360

Commit message: FIN PLACA 2
FIN PLACA 2
Parts:
- removed J14: Conn_01x10_Pin, Connector_PinSocket_2.54mm:PinSocket_1x10_P2.54mm_Vertical
- removed JP1: Conn_01x10_Pin, Connector_PinHeader_2.54mm:PinHeader_1x10_P2.54mm_Vertical
- added J17: VCC, Connector_PinSocket_2.00mm:PinSocket_1x01_P2.00mm_Vertical, F.Cu at (215.2, 72.0)
- added J18: OUT, Connector_PinSocket_2.00mm:PinSocket_1x01_P2.00mm_Vertical, F.Cu at (211.1, 73.5)
- added J19: GND, Connector_PinSocket_2.00mm:PinSocket_1x01_P2.00mm_Vertical, F.Cu at (196.4, 80.0)
- added J20: Conn_01x08_Pin, Connector_PinHeader_2.54mm:PinHeader_1x08_P2.54mm_Vertical, F.Cu at (242.7, 54.0)
- added J21: Conn_01x08_Pin, Connector_PinSocket_2.54mm:PinSocket_1x08_P2.54mm_Vertical, F.Cu at (69.5, 147.1)
- moved RV1 206.3 mm to (268.3, 105.3)
- moved R9 113.3 mm to (129.9, 50.2), turned to 0 degrees
- moved R9!1 110.7 mm to (130.9, 53.7), turned to 0 degrees
- moved R11 110.2 mm to (129.9, 60.2), turned to 0 degrees
- moved R11!1 108.6 mm to (130.4, 64.7), turned to 0 degrees
- moved R7 94.7 mm to (131.9, 68.6), turned to 0 degrees
- moved R7!1 92.8 mm to (131.9, 72.6), turned to 0 degrees
- moved JP3 92.6 mm to (122.5, 67.3), turned to 0 degrees
- moved R8 87.2 mm to (150.2, 55.5), turned to 0 degrees
- moved R8!1 85.4 mm to (147.4, 60.0), turned to 0 degrees
- moved R13 84.4 mm to (193.3, 78.2)
- moved JP2 82.5 mm to (127.5, 71.6), turned to 0 degrees
- moved R12 71.7 mm to (132.1, 103.4), turned to 0 degrees
- moved R10!1 68.9 mm to (132.4, 95.9), turned to 0 degrees
- moved R10 68.1 mm to (132.6, 91.9), turned to 0 degrees
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Connections:
- RV1 pad 1: VCCSw -> unconnected-(RV1-Pad1)
- RV1 pad 2: /PinPotOut1 -> unconnected-(RV1-Pad2)
- RV1 pad 3: GNDSw -> unconnected-(RV1-Pad3)
Routing:
- net /PinPotOut1: track 27.2 -> 0.00 mm
- net VCCSw: track 16.3 -> 0.00 mm
- net /OscOut1: track 42.9 -> 40.5 mm
Other:
- board size 70.6 x 51.2 mm -> 69.2 x 51.4 mm

Commit message: lindo avance placa principal
Parts:
- moved R11 101.9 mm to (174.8, 151.8), turned to 90 degrees
- moved J20 100.0 mm to (223.4, 152.1)
- moved R11!1 92.6 mm to (178.0, 144.1), turned to -90 degrees
- moved JP3 91.5 mm to (157.0, 152.0), turned to 180 degrees
- moved JP2 89.0 mm to (163.1, 153.2), turned to 180 degrees
- moved R9!1 88.6 mm to (173.2, 131.6), turned to 90 degrees
- moved R9 84.2 mm to (170.4, 124.0), turned to -90 degrees
- moved R7!1 79.1 mm to (184.8, 131.6), turned to 90 degrees
- moved R8!1 78.2 mm to (178.9, 131.6), turned to 90 degrees
- moved J17 77.0 mm to (253.8, 138.7)
- moved J19 77.0 mm to (234.9, 146.6)
- moved J18 77.0 mm to (249.6, 140.2)
- moved R13 77.0 mm to (231.8, 144.8)
- moved R7 74.4 mm to (181.8, 123.9), turned to -90 degrees
- moved R8 73.1 mm to (175.9, 123.9), turned to -90 degrees
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Routing:
- net GND: track 0.00 -> 113.3 mm
- net VCC: track 0.00 -> 104.0 mm
- net /PinCOut: track 0.00 -> 71.7 mm
- net /PinBOut: track 0.00 -> 62.1 mm
- net /PinAOut: track 0.00 -> 53.4 mm
- net /PinDIn: track 0.00 -> 47.5 mm
- net /PinEIn: track 0.00 -> 46.3 mm
- net /PinFIn: track 0.00 -> 46.2 mm
- net /PinAIn: track 0.00 -> 35.4 mm
- net /PinBIn: track 0.00 -> 34.5 mm
- net /PinCIn: track 0.00 -> 33.8 mm
- net /PinFOut: track 0.00 -> 23.5 mm
- net /PinEOut: track 0.00 -> 18.1 mm
- net /PinDOut: track 0.00 -> 11.2 mm
- net /PinC6: track 30.3 -> 35.4 mm
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
Commit message: avance piolita en placa principal
Parts:
- moved RV1 124.1 mm to (145.2, 120.8), turned to 90 degrees
- moved U10 35.3 mm to (198.4, 140.6), turned to 90 degrees
- moved J_USB1 28.8 mm to (210.5, 123.8)
- moved U2 19.2 mm to (201.8, 149.2), turned to 0 degrees
- moved J_JACK1 19.1 mm to (200.0, 128.8), turned to -90 degrees
- moved R2 13.5 mm to (212.7, 138.8)
- moved R1 13.5 mm to (212.7, 135.7)
- moved R3 13.5 mm to (212.7, 141.9)
- moved R4 13.5 mm to (212.7, 145.1)
- moved R5 13.5 mm to (212.7, 148.2)
- moved R6 13.5 mm to (212.7, 151.4)
Routing:
- net VCC: track 104.0 -> 82.2 mm

Commit message: revision final
Parts:
- J_USB1: moved to B.Cu
- moved J17 46.7 mm to (207.8, 147.0)
- moved J18 43.0 mm to (207.8, 150.6)
- moved R13 28.7 mm to (204.7, 154.3)
- moved J19 28.3 mm to (207.7, 154.5)
- moved U10 14.7 mm to (194.0, 154.5)
- moved U2 10.0 mm to (202.0, 139.2)
- moved J_JACK1 2.15 mm to (200.8, 130.8)
- moved J_USB1 0.87 mm to (211.4, 123.9), turned to 0 degrees
- moved R3 0.61 mm to (212.6, 142.6)
- moved R1 0.61 mm to (212.6, 136.2)
- moved R2 0.61 mm to (212.6, 139.4)
- moved R4 0.61 mm to (212.6, 145.7)
- moved R5 0.61 mm to (212.6, 148.8)
- moved R6 0.61 mm to (212.6, 152.0)
Connections:
- J_USB1 pad 1: VCC_nreg -> VCC
Routing:
- net GND: track 113.3 -> 236.9 mm
- net VCC: track 82.2 -> 146.8 mm
- net /OscOut: track 0.00 -> 45.9 mm
- net /PinPot1: track 0.00 -> 16.2 mm
- net VCC_nreg: track 0.00 -> 15.7 mm
- net Net-(U10-TR): track 0.00 -> 9.33 mm
- net /PinPot3: track 0.00 -> 6.95 mm
- net /PinR1: track 0.00 -> 5.02 mm
- net /PinR2: track 0.00 -> 4.48 mm
- net /PinR3: track 0.00 -> 4.04 mm
- net /PinR4: track 0.00 -> 3.99 mm
- net /PinR5: track 0.00 -> 3.74 mm
- net /PinR6: track 0.00 -> 3.27 mm
- net /PinFIn: track 46.2 -> 47.7 mm
- net /PinAIn: track 35.4 -> 33.9 mm
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Other:
- board size 69.2 x 51.4 mm -> 204.7 x 59.5 mm

Commit message: hecho plano de masa y tornillos
Parts:
- removed RV1: 5K, Potentiometer_THT:Potentiometer_Omeg_PC16BU_Horizontal
- added REF**: MountingHole_2.2mm_M2, MountingHole:MountingHole_2.2mm_M2, F.Cu at (132.7, 82.5)
- added REF**: MountingHole_2.2mm_M2, MountingHole:MountingHole_2.2mm_M2, F.Cu at (268.3, 128.2)
- added REF**: MountingHole_2.2mm_M2, MountingHole:MountingHole_2.2mm_M2, F.Cu at (248.8, 128.2)
- added REF**: MountingHole_2.2mm_M2, MountingHole:MountingHole_2.2mm_M2, F.Cu at (45.4, 17.3)
- added REF**: MountingHole_2.2mm_M2, MountingHole:MountingHole_2.2mm_M2, F.Cu at (233.0, 89.2)
- added REF**: MountingHole_2.2mm_M2, MountingHole:MountingHole_2.2mm_M2, F.Cu at (199.4, 120.9)
- added REF**: MountingHole_2.2mm_M2, MountingHole:MountingHole_2.2mm_M2, F.Cu at (152.2, 127.5)
- added REF**: MountingHole_2.2mm_M2, MountingHole:MountingHole_2.2mm_M2, F.Cu at (170.1, 89.2)
- added REF**: MountingHole_2.2mm_M2, MountingHole:MountingHole_2.2mm_M2, F.Cu at (268.1, 83.5)
- added REF**: MountingHole_2.2mm_M2, MountingHole:MountingHole_2.2mm_M2, F.Cu at (152.2, 82.5)
- added REF**: MountingHole_2.2mm_M2, MountingHole:MountingHole_2.2mm_M2, F.Cu at (96.1, 17.6)
- added REF**: MountingHole_2.2mm_M2, MountingHole:MountingHole_2.2mm_M2, F.Cu at (248.8, 83.5)
- added REF**: MountingHole_2.2mm_M2, MountingHole:MountingHole_2.2mm_M2, F.Cu at (205.7, 89.2)
- added REF**: MountingHole_2.2mm_M2, MountingHole:MountingHole_2.2mm_M2, F.Cu at (132.7, 127.5)
- moved J15 193.6 mm to (258.8, 129.0)
- moved R14 185.6 mm to (248.6, 89.6), turned to 45 degrees
- moved C6 185.3 mm to (255.8, 122.0)
- moved C1 185.3 mm to (255.9, 89.7)
- moved C2 185.3 mm to (255.9, 96.2)
- moved C3 185.3 mm to (255.9, 102.7)
- moved C4 185.3 mm to (255.9, 109.2)
- moved C5 185.3 mm to (255.9, 115.5)
- moved J1 185.3 mm to (252.6, 90.9)
- moved J2 185.3 mm to (252.6, 97.2)
- moved J21 185.3 mm to (248.5, 94.5)
- moved J3 185.3 mm to (252.6, 103.6)
- moved J4 185.3 mm to (252.6, 109.9)
- moved J5 185.3 mm to (252.6, 116.4)
- moved J6 185.3 mm to (252.6, 123.2)
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Routing:
- net GND: track 236.9 -> 120.4 mm
- net unconnected-(J_USB1-Shield-Pad6): track 0.00 -> 12.6 mm
- net /PinC2: track 23.8 -> 15.7 mm
- net GNDSw: track 181.6 -> 175.7 mm
- net /PinC5: track 30.1 -> 25.0 mm
- net /PinC6: track 35.4 -> 30.5 mm
- net /PinC1: track 23.0 -> 18.7 mm
- net /PinC4: track 27.4 -> 23.2 mm
- net /OscOut1: track 36.9 -> 33.3 mm
- net /PinC3: track 22.8 -> 19.4 mm
- net VCC_nreg: track 15.7 -> 18.4 mm
- net /PinDOut1: track 45.9 -> 44.0 mm
- net /PinAOut1: track 35.6 -> 33.7 mm
- net /PinEOut1: track 40.5 -> 39.0 mm
- net VCCLed: track 70.2 -> 68.8 mm
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- added copper zone on B.Cu, net (none)
- added copper zone on B.Cu, net GND
- added copper zone on B.Cu, net GNDSw
Other:
- board size 204.7 x 59.5 mm -> 140.6 x 50.8 mm
